Commit message: Minor typo

File: uuv_gazebo_plugins/uuv_gazebo_ros_plugins/test/models/thrusters/model.xacro (robot description, xacro)
@@ -19,5 +19,5 @@
 <robot name="rexrov" xmlns:xacro="http://www.ros.org/wiki/xacro" >
   <xacro:include filename="$(find uuv_gazebo_ros_plugins)/urdf/thruster_snippets.xacro"/>
-  <xacro:property name="prop_mesh_file" value="file://$(find uuv_descriptions)/mesh/prop.dae"/>
+  <xacro:property name="prop_mesh_file" value="file://$(find uuv_descriptions)/meshes/prop.dae"/>
   <xacro:macro name="box_inertial" params="x y z mass *origin">
     <inertial>
