Commit message: Added missing parameter to dvl sensor.

File: uuv_sensor_plugins/uuv_sensor_ros_plugins/urdf/dvl_snippets.xacro (robot description, xacro)
@@ -71,5 +71,5 @@
     </xacro:dvl_plugin_macro>
   </xacro:macro>
-  <xacro:macro name="dvl_single_sonar" params="namespace suffix index pitch yaw update_rate">
+  <xacro:macro name="dvl_single_sonar" params="namespace suffix index pitch yaw update_rate topic">
     <link name="${namespace}/dvl${suffix}_sonar${index}_link">
       <inertial>
@@ -161,17 +161,17 @@
     <xacro:dvl_single_sonar
       namespace="${namespace}" suffix=""
-      index="0" pitch="-0.52" yaw="0.0" update_rate="${update_rate}">
-    </xacro:dvl_single_sonar>
-    <xacro:dvl_single_sonar
-      namespace="${namespace}" suffix=""
-      index="1" pitch="0" yaw="0.52" update_rate="${update_rate}">
-    </xacro:dvl_single_sonar>
-    <xacro:dvl_single_sonar
-      namespace="${namespace}" suffix=""
-      index="2" pitch="0.52" yaw="0.0" update_rate="${update_rate}">
-    </xacro:dvl_single_sonar>
-    <xacro:dvl_single_sonar
-      namespace="${namespace}" suffix=""
-      index="3" pitch="0.0" yaw="-0.52" update_rate="${update_rate}">
+      index="0" pitch="-0.52" yaw="0.0" update_rate="${update_rate}" topic="${topic}">
+    </xacro:dvl_single_sonar>
+    <xacro:dvl_single_sonar
+      namespace="${namespace}" suffix=""
+      index="1" pitch="0" yaw="0.52" update_rate="${update_rate}" topic="${topic}">
+    </xacro:dvl_single_sonar>
+    <xacro:dvl_single_sonar
+      namespace="${namespace}" suffix=""
+      index="2" pitch="0.52" yaw="0.0" update_rate="${update_rate}" topic="${topic}">
+    </xacro:dvl_single_sonar>
+    <xacro:dvl_single_sonar
+      namespace="${namespace}" suffix=""
+      index="3" pitch="0.0" yaw="-0.52" update_rate="${update_rate}" topic="${topic}">
     </xacro:dvl_single_sonar>
     <gazebo>
